File: ATO-Encoder-PCB/ATO-Encoder-PCB.kicad_sch (KiCad schematic)
At the start: 0 parts

Commit message: Schematic complete and PCB layout in progress. Need to select specific component and update footprints. Need to update resistances for leds. Need to add power LED. Need to reorganize to shrink PCB size.
Parts:
- added C1, C3: 0.1uF, Capacitor_SMD:C_0805_2012Metric, symbol rdsData-eagle-import:CAP
- added C2, C8: 4700pF, Capacitor_SMD:C_0805_2012Metric, symbol rdsData-eagle-import:CAP
- added D1, D2, D3: LED, LED_SMD:LED_0201_0603Metric, symbol Device:LED
- added IC1, IC3: MCP2561-H_P, Package_DIP:DIP-8_W7.62mm, symbol rdsData-eagle-import:MCP2561-H_P
- added J1: DE9_Socket, Connector_Dsub:DSUB-9_Socket_Vertical_P2.77x2.84mm_MountingHoles, symbol Connector:DE9_Socket
- added J2: Conn_01x06, Connector_PinHeader_2.54mm:PinHeader_1x06_P2.54mm_Vertical, symbol Connector_Generic:Conn_01x06
- added J3, J4, J5, J6: B2B-XH-A, BoardToCable_2PinMale:JST_B2B-XH-A, symbol Digikey Components:B2B-XH-A
- added JP1, JP2: PINHD-1X24, Connector_PinHeader_2.54mm:PinHeader_1x24_P2.54mm_Vertical, symbol rdsData-eagle-import:PINHD-1X24
- added R1, R2, R3: 120R, Resistor_SMD:R_0805_2012Metric, symbol Device:R_US
- added R10, R5: 300Ohm, Resistor_SMD:R_0805_2012Metric, symbol rdsData-eagle-import:RES
- added R11, R12, R7, R8: 60Ohm, Resistor_SMD:R_0805_2012Metric, symbol rdsData-eagle-import:RES
- added R4, R6, R9: 330R, Resistor_SMD:R_0805_2012Metric, symbol Device:R_US
- added U$1: TEENSY4-1, Teensy4.1:Teensy 4.1, symbol rdsData-eagle-import:TEENSY4-1
- added U1: ~, Package_DFN_QFN:TQFN-32-1EP_5x5mm_P0.5mm_EP3.1x3.1mm, symbol ATO Breakout Components:MAX14890E
Connections:
- new net: C2.2, R5.2, R7.1, R8.2
- new net: JP2.10, U$1.P38 (SDA1/TX4/A3/P17)
- new net: JP2.11, U$1.P37 (SCL1/RX4/A2/P16)
- new net: JP2.12, U$1.P36 (PWM/S/PDIF-IN/RX3/A1/P15)
- new net: JP2.13, U$1.P35 (PWM/S/PDIF-OUT/TX3/A0/P14)
- new net: JP2.16, U$1.P32 (A17/P41)
- new net: JP2.17, U$1.P31 (A16/P40)
- new net: JP2.18, U$1.P30 (OUT1A/MISO1/A15/P39)
- new net: JP2.19, U$1.P29 (IN1/CS1/A14/P38)
- new net: JP2.20, U$1.P28 (CS/PWM/P37)
- new net: JP2.21, U$1.P27 (CS/PWM/P36)
- new net: JP2.22, U$1.P26 (TX8/P35)
- new net: JP2.23, U$1.P25 (RX8/P34)
- new net: JP2.24, U$1.P24 (MCLK2/PWM/P33)
- new net: JP2.4, U$1.P44 (PWM/MCLK1/CRX1/A9/P23)
- new net: JP2.5, U$1.P43 (PWM/CTX1/A8/P22)
- new net: JP2.6, U$1.P42 (BLCK1/RX5/A7/P21)
- new net: JP1.10, U$1.P9 (P8/PWM/IN1/TX2)
- new net: JP1.11, U$1.P10 (P9/PWM/OUT1C)
- new net: JP1.16, U$1.P15 (P24/PWM/SCL2/TX6/A10)
- new net: JP1.17, U$1.P16 (P25/PWM/SDA2/RX6/A11)
- new net: JP1.18, U$1.P17 (P26/MOSI1/A12)
- new net: JP1.19, U$1.P18 (P27/SCK1/A13)
- new net: JP1.20, U$1.P19 (P28/PWM/RX7)
- new net: JP1.21, U$1.P20 (P29/PWM/TX7)
- new net: JP1.24, U$1.P23 (P32/OUT1B)
- new net: JP1.7, U$1.P6 (P5/PWM/IN2)
- new net: JP1.8, U$1.P7 (P6/PWM/OUT1D)
- new net: JP1.9, U$1.P8 (P7/PWM/OUT1A/RX2)
- new net: IC3.5 (SPLIT), R10.1
- new net: J1.2, R1.2, U1.25 (Z)
- new net: J1.3, R2.1, U1.9 (B)
- new net: J1.4, R3.1, U1.32 (A)
- new net: J1.6, R1.1, U1.26 (~{Z})
- new net: J1.7, R2.2, U1.10 (~{B})
- new net: J1.8, R3.2, U1.31 (~{A})
- new net: D1.1 (K), R4.2
- new net: R9.1, U1.2 (~{AFAULT})
- new net: R4.1, U1.20 (~{ZFAULT})
- new net: R6.1, U1.21 (~{BFAULT})
- new net: D2.1 (K), R6.2
- new net: C8.2, R10.2, R11.1, R12.2
- new net: IC1.5 (SPLIT), R5.1
- new net: D3.1 (K), R9.2
- new net +5V: C1.2, C3.1, D1.2 (A), D2.2 (A), D3.2 (A), IC1.3 (VDD), IC3.3 (VDD), J1.5, JP2.1, U$1.P47 (VIN), U1.27 (V_{CC})
- new net 3v3: J2.6 (Pin_6), JP1.15, JP2.3, U$1.P14 (3V3@1), U$1.P45 (3V3@2), U1.22 (V_{L})
- new net AO: JP1.5, U$1.P4 (P3/PWM/LRCLK2), U1.1 (AO)
- new net BO: JP1.4, U$1.P3 (P2/PWM/OUT2), U1.8 (BO)
- new net CANH2: IC1.7 (CANH), J3.1, J5.1, R7.2
- new net CANH3: IC3.7 (CANH), J4.1, J6.1, R11.2
- new net CANL2: IC1.6 (CANL), J3.2, J5.2, R8.1
- new net CANL3: IC3.6 (CANL), J4.2, J6.2, R12.1
- new net CLK: JP2.14, U$1.P34 (PWM/SCK/(LED)P13), U1.4 (~{CS})
- new net CRX2: IC1.4 (RXD), JP1.2, U$1.P1 (P0/PWM/CRX2/CS1/RX1)
- new net CRX3: IC3.4 (RXD), JP1.22, U$1.P21 (P30/CRX3)
- new net CS: JP1.12, U$1.P11 (P10/PWM/MQSR/CS), U1.3 (SDO)
- new net CTX2: IC1.1 (TXD), JP1.3, U$1.P2 (P1/PWM/CTX2/MISO1/TX1)
- new net CTX3: IC3.1 (TXD), JP1.23, U$1.P22 (P31/CTX3)
- new net Encoder Fault: U1.7 (~{IRQ})
- new net GND: C1.1, C2.1, C3.2, C8.1, IC1.2 (VSS), IC1.8 (STBY), IC3.2 (VSS), IC3.8 (STBY), J1.1, J1.9, J2.4 (Pin_4), JP1.1, JP2.15, JP2.2, U$1.P0 (GND@1), U$1.P33 (GND@2), U$1.P46 (GND@3), U1.11 (GND)
- new net SCL: J2.3 (Pin_3), JP2.8, U$1.P40 (PWM/SCL/A5/P19)
- new net SDA: J2.2 (Pin_2), JP2.9, U$1.P39 (PWM/SDA/A4/P18)
- new net SDI: JP1.13, U$1.P12 (P11/PWM/CTX1/MOSI), U1.6 (SDI)
- new net SDO: JP1.14, U$1.P13 (P12/PWM/MQSL/MISO), U1.5 (CLK)
- new net SPI: JP2.7, U$1.P41 (LRCLK1/TX5/A6/P20), U1.23 (SPI)
- new net ZO: JP1.6, U$1.P5 (P4/PWM/BCLK2), U1.24 (ZO)
Other:
- note added: "CAN Transciever Circuit"
- note added: "Load Cell Amplifier Connection"
- note added: "RS-422 Quadrature Reciever Circuit"
- note added: "Teensy 4.1 Circuit"

Commit message: PBC is ready for manufacture
Parts:
- removed C1: 0.1uF, Capacitor_SMD:C_0805_2012Metric, symbol rdsData-eagle-import:CAP
- removed C2: 4700pF, Capacitor_SMD:C_0805_2012Metric, symbol rdsData-eagle-import:CAP
- removed IC1: MCP2561-H_P, Package_DIP:DIP-8_W7.62mm, symbol rdsData-eagle-import:MCP2561-H_P
- removed J3, J5: B2B-XH-A, BoardToCable_2PinMale:JST_B2B-XH-A, symbol Digikey Components:B2B-XH-A
- removed R5: 300Ohm, Resistor_SMD:R_0805_2012Metric, symbol rdsData-eagle-import:RES
- removed R7, R8: 60Ohm, Resistor_SMD:R_0805_2012Metric, symbol rdsData-eagle-import:RES
- added C3, C4: 3.3uF, Capacitor_SMD:C_0805_2012Metric, symbol rdsData-eagle-import:CAP
- added D4: LED, LED_THT:LED_D3.0mm, symbol Device:LED
- added J5: Screw_Terminal_01x02, TerminalBlock:TerminalBlock_MaiXu_MX126-5.0-02P_1x02_P5.00mm, symbol Connector:Screw_Terminal_01x02
- added R10: 150R, Resistor_SMD:R_0805_2012Metric, symbol Device:R_US
- D1, D2, D3: footprint LED_SMD:LED_0201_0603Metric -> LED_THT:LED_D3.0mm
- R4, R6, R9: value 330R -> 150R
- renumbered C3 to C1, C8 to C2, IC3 to IC1, J6 to J2, J4 to J3, J2 to J4, R10 to R5, R11 to R7, R12 to R8
Connections:
- net +5V: now also D4.2 (A), J5.1 (Pin_1)
- net 3v3: now also C3.2, C4.2
- net AO: now also JP1.8, U$1.P7 (P6/PWM/OUT1D); no longer JP1.5, U$1.P4 (P3/PWM/LRCLK2)
- net BO: now also JP1.9, U$1.P8 (P7/PWM/OUT1A/RX2); no longer JP1.4, U$1.P3 (P2/PWM/OUT2)
- net Encoder Fault: now also JP1.10, U$1.P9 (P8/PWM/IN1/TX2)
- net GND: now also C3.1, C4.1, J5.2 (Pin_2), R10.2
- net SPI: now also JP1.18, U$1.P17 (P26/MOSI1/A12); no longer JP2.7, U$1.P41 (LRCLK1/TX5/A6/P20)
- net ZO: now also JP1.17, U$1.P16 (P25/PWM/SDA2/RX6/A11); no longer JP1.6, U$1.P5 (P4/PWM/BCLK2)
- new net: JP2.7, U$1.P41 (LRCLK1/TX5/A6/P20)
- new net: JP1.4, U$1.P3 (P2/PWM/OUT2)
- new net: JP1.5, U$1.P4 (P3/PWM/LRCLK2)
- new net: JP1.6, U$1.P5 (P4/PWM/BCLK2)
- new net: D4.1 (K), R10.1
